Commit message: Added other US sensor, but need to set correct position

File: b4-description/urdf/b4.urdf (robot description, URDF)
Before this commit: robot B4, 4 links, 3 joints
Links:
- removed link uSonarRange_topic
- added link topicSonarRangeCenter; visual box size=0.045 0.02 0.015
- added link topicSonarRangeLeft; visual box size=0.045 0.02 0.015
- added link topicSonarRangeRight; visual box size=0.045 0.02 0.015
Joints:
- removed joint base_link_to_base_uSonarRange_topic
- added joint base_link_to_topicSonarRangeCenter: type fixed, parent base_link, child topicSonarRangeCenter, origin xyz=0.09 0 0.08 rpy=0 0 0
- added joint base_link_to_topicSonarRangeLeft: type fixed, parent base_link, child topicSonarRangeLeft, origin xyz=0.09 0 0.08 rpy=0 0 0
- added joint base_link_to_topicSonarRangeRight: type fixed, parent base_link, child topicSonarRangeRight, origin xyz=0.09 0 0.08 rpy=0 0 0

Commit message: correct the position of USsensors

File: b4-description/urdf/b4.urdf (robot description, URDF)
Before this commit: robot B4, 6 links, 5 joints
Links:
- link base_link: geometry visual cylinder length=0.200 radius=0.1
- link topicSonarRangeCenter: geometry visual box size=0.015 0.045 0.020
- link topicSonarRangeLeft: geometry visual box size=0.015 0.045 0.020
- link topicSonarRangeRight: geometry visual box size=0.015 0.045 0.020
Joints:
- joint base_link_to_topicSonarRangeCenter: origin xyz=0.09 0 0.08 rpy=0 0 0 -> xyz=0.095 0 0.106 rpy=0 0 0
- joint base_link_to_topicSonarRangeLeft: origin xyz=0.09 0 0.08 rpy=0 0 0 -> xyz=0.085 -0.040 0.08 rpy=0 0 -0.523599
- joint base_link_to_topicSonarRangeRight: origin xyz=0.09 0 0.08 rpy=0 0 0 -> xyz=0.085 0.040 0.08 rpy=0 0 0.523599
